File: eagle/ESPNTPServer/ESPNTPServer.sch (EAGLE design)
At the start: 23 parts, among them J1 POWER_JACK, U1 MCP1825/DC

Commit message: Change power supply from linar to Switch
Parts:
- removed C4: 100uf, rcl:CPOL-EUE2.5-5
- removed U1: MCP1825/DC, MCP1825:MCP1825/DC
- added C5: 470 pf, resistor:C-EUC1206
- added C7: 470мкф, resistor:CPOL-EUE3.5-8
- added D1: MBRS130LT3, diode:MBRS130LT3
- added IC1: MC34063AD, mc34063:MC34063AD
- added J2: POWER_JACK, ESPNTPServer:POWER_JACK
- added L1: 220 uH, inductor-neosid:SD12K-82
- added R10: 1.2k, resistor:R-EU_M1206
- added R11: 10k, resistor:R-EU_M1206
- added R8: 3.6k, resistor:R-EU_M1206
- added R9: 0.33, resistor:R-EU_0411/3V
- added SJ1: (no value), jumper:SJ
- C1: value 10uf -> (none); device rcl:C-EU050-025X075 -> resistor:C-EUC1206
- C3: value 10uf -> 470мкф; device rcl:C-EU050-025X075 -> resistor:CPOL-EUE3.5-8
- J1: value POWER_JACK -> DM3AT-SF-PEJM5; device ESPNTPServer:POWER_JACK -> connector:DM3AT-SF-PEJM5
- R1, R2, R3, R4, R5, R6, R7: device rcl:R-EU_0204/2V -> resistor:R-EU_M1206
Connections:
- new net N$2: IC1.DC, IC1.IS, IC1.SWC, R9.1
- new net N$3: C5.1, IC1.TC
- new net N$5: D1.C, IC1.SWE, L1.1
- new net N$6: IC1.FB, R10.1, R8.2
- new net SD_CLK: J1.CLK, MDL1.SCLK
- new net SD_CMD: J1.CMD/MOSI, MDL1.CS0
- new net SD_D0: J1.DATA0/MISO, MDL1.MISO
- new net SD_D1: J1.DATA1/RSV, MDL1.MOSI
- new net SD_D2: J1.DATA2/NC, MDL1.GPIO9
- new net SD_D3: J1.DATA3-CD/CS_N, MDL1.GPIO10
- new net SD_DET: J1.B, R11.2, SJ1.2
- new net SD_DET_N: MDL1.GPIO16, SJ1.1
- net GND: now also C1.2, C3.-, C5.2, C7.-, D1.A, IC1.GND, J1.A, J2.GND, R10.2; no longer C1.1, C3.2, C4.-, U1.GND
- net VCC: now also C1.1, C7.+, J1.VCC, JP3.5, L1.2, R11.1, R8.1; no longer C3.1, C4.+, U1.VOUT
- net VIN: now also C3.+, IC1.VCC, J2.PWR, R9.2; no longer C1.2, J1.PWR, JP3.5, U1.!SHDN, U1.VIN
Other:
- moved on the sheet: C1
